File: TKL2019/_autosave-TKL2019.kicad_pcb (KiCad board)
At the start: 2 copper layers, 152 parts, among them J1 USB_mini_micro_B, J2 KEYSW, K1 KEYSW, M1 KEYSW, P1 KEYSW, Q1 KEYSW, SW1 SW_PUSH, T1 KEYSW, U1 ATMEGA32U4, U2 KEYSW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

Commit message: a lot of progress
Parts:
- BACKSPACE1: footprint Button_Switch_Keyboard:SW_Cherry_MX_2.00u_Plate -> Button_Switch_Keyboard:SW_Cherry_MX_2.00u_PCB
- C1, C2, C3, C4, C5, C6, C7, C8: footprint Capacitor_SMD:C_0805_2012Metric_Pad1.15x1.40mm_HandSolder -> oldstuff:C_0805_HandSoldering
- ENTER1, SHIFT1: footprint Button_Switch_Keyboard:SW_Cherry_MX_2.25u_Plate -> Button_Switch_Keyboard:SW_Cherry_MX_2.25u_PCB
- R1, R2, R3, R4: footprint Resistor_SMD:R_0805_2012Metric_Pad1.15x1.40mm_HandSolder -> oldstuff:R_0805_HandSoldering
- SPACE1: footprint Button_Switch_Keyboard:SW_Cherry_MX_6.25u_Plate -> Button_Switch_Keyboard:SW_Cherry_MX_6.25u_PCB
- moved R1 91.5 mm to (120.6, 131.7)
- moved C2 91.5 mm to (132.5, 133.8), turned to 90 degrees
- moved X1 85.1 mm to (137.0, 133.8), turned to 180 degrees
- moved C1 79.4 mm to (141.3, 133.8), turned to 270 degrees
- moved SW1 78.9 mm to (126.0, 131.9)
- moved U1 68.7 mm to (177.7, 113.0)
- moved R2 66.4 mm to (186.7, 113.0), turned to 270 degrees
- moved R4 64.6 mm to (135.4, 129.2), turned to 180 degrees
- moved C6 63.1 mm to (144.6, 133.8), turned to 270 degrees
- moved C7 62.8 mm to (168.7, 108.0), turned to 90 degrees
- moved C5 58.8 mm to (168.6, 118.5), turned to 90 degrees
- moved C3 57.9 mm to (186.7, 108.0), turned to 90 degrees
- moved R3 56.9 mm to (142.9, 129.3), turned to 180 degrees
- moved C8 56.1 mm to (168.6, 113.4), turned to 90 degrees
- moved C4 44.1 mm to (186.7, 118.0), turned to 90 degrees
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