File: TKL2019/TKL2019.kicad_pcb (KiCad board)
At the start: 2 copper layers, 152 parts, among them J1 USB_mini_micro_B, J2 KEYSW, K1 KEYSW, M1 KEYSW, P1 KEYSW, Q1 KEYSW, SW1 SW_PUSH, T1 KEYSW, U1 ATMEGA32U4, U2 KEYSW, X1 XTAL_GND, X2 KEYSW, Y1 KEYSW

Commit message: a lot of progress
Parts:
- BACKSPACE1: footprint Button_Switch_Keyboard:SW_Cherry_MX_2.00u_Plate -> Button_Switch_Keyboard:SW_Cherry_MX_2.00u_PCB
- C1, C2, C3, C4, C5, C6, C7, C8: footprint Capacitor_SMD:C_0805_2012Metric_Pad1.15x1.40mm_HandSolder -> oldstuff:C_0805_HandSoldering
- ENTER1, SHIFT1: footprint Button_Switch_Keyboard:SW_Cherry_MX_2.25u_Plate -> Button_Switch_Keyboard:SW_Cherry_MX_2.25u_PCB
- R1, R2, R3, R4: footprint Resistor_SMD:R_0805_2012Metric_Pad1.15x1.40mm_HandSolder -> oldstuff:R_0805_HandSoldering
- SPACE1: footprint Button_Switch_Keyboard:SW_Cherry_MX_6.25u_Plate -> Button_Switch_Keyboard:SW_Cherry_MX_6.25u_PCB
- moved R1 91.5 mm to (120.6, 131.7)
- moved C2 91.5 mm to (132.5, 133.8), turned to 90 degrees
- moved X1 85.1 mm to (137.0, 133.8), turned to 180 degrees
- moved C1 79.4 mm to (141.3, 133.8), turned to 270 degrees
- moved SW1 78.9 mm to (126.0, 131.9)
- moved U1 68.7 mm to (177.7, 113.0)
- moved R2 66.4 mm to (186.7, 113.0), turned to 270 degrees
- moved R4 64.6 mm to (135.4, 129.2), turned to 180 degrees
- moved C6 63.1 mm to (144.6, 133.8), turned to 270 degrees
- moved C7 62.8 mm to (168.7, 108.0), turned to 90 degrees
- moved C5 58.8 mm to (168.6, 118.5), turned to 90 degrees
- moved C3 57.9 mm to (186.7, 108.0), turned to 90 degrees
- moved R3 56.9 mm to (142.9, 129.3), turned to 180 degrees
- moved C8 56.1 mm to (168.6, 113.4), turned to 90 degrees
- moved C4 44.1 mm to (186.7, 118.0), turned to 90 degrees
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
Commit message: changed some stuff
Parts:
- added REF**: MountingHole_2.2mm_M2, MountingHole:MountingHole_2.2mm_M2, F.Cu at (249.8, 153.6)
- added REF**: MountingHole_2.2mm_M2, MountingHole:MountingHole_2.2mm_M2, F.Cu at (284.2, 113.1)
- added REF**: MountingHole_2.2mm_M2, MountingHole:MountingHole_2.2mm_M2, F.Cu at (230.8, 152.9)
- added REF**: MountingHole_2.2mm_M2, MountingHole:MountingHole_2.2mm_M2, F.Cu at (215.5, 157.6)
- added REF**: MountingHole_2.2mm_M2, MountingHole:MountingHole_2.2mm_M2, F.Cu at (216.4, 138.1)
- J1: footprint keyboard_parts:USB_miniB_hirose_5S8 -> SamacSys_Parts:1734035-2USB; moved to B.Cu
- moved ESC1 11.3 mm to (24.6, 42.0), turned to 180 degrees
- moved NO1 11.3 mm to (43.6, 42.0), turned to 180 degrees
- moved D67 9.90 mm to (277.2, 122.1), turned to 180 degrees
- moved D1 8.75 mm to (31.6, 46.0), turned to 180 degrees
- moved J1 4.16 mm to (38.8, 32.7), turned to 270 degrees
- moved SW1 0.86 mm to (126.9, 131.8)

Commit message: bruh
Parts:
- removed REF** (x4): MountingHole_2.2mm_M2, MountingHole:MountingHole_2.2mm_M2
- added D70: LED, LED_THT:LED_D3.0mm, F.Cu at (32.9, 80.2)
- added MH2: MountingHole_2.2mm_M2, MountingHole:MountingHole_2.2mm_M2, F.Cu at (278.0, 56.0)
- added MH3: MountingHole_2.2mm_M2, MountingHole:MountingHole_2.2mm_M2, F.Cu at (146.1, 75.2)
- added MH4: MountingHole_2.2mm_M2, MountingHole:MountingHole_2.2mm_M2, F.Cu at (42.5, 113.1)
- added MH5: MountingHole_2.2mm_M2, MountingHole:MountingHole_2.2mm_M2, F.Cu at (203.9, 113.4)
- added MH6: MountingHole_2.2mm_M2, MountingHole:MountingHole_2.2mm_M2, F.Cu at (284.2, 113.1)
- added R10: 22, oldstuff:R_0805_HandSoldering, B.Cu at (58.4, 91.4)
- added R6: 22, oldstuff:R_0805_HandSoldering, B.Cu at (53.4, 96.4)
- added R7: 22, oldstuff:R_0805_HandSoldering, B.Cu at (55.9, 91.4)
- added R8: 22, oldstuff:R_0805_HandSoldering, B.Cu at (55.9, 96.4)
- added R9: 22, oldstuff:R_0805_HandSoldering, B.Cu at (58.4, 96.4)
- C1, C2, C3, C4, C5, C6, C7, C8, D1, D10, D11, D12, D13, D14, D15, D16, D17, D18, D19, D2, D20, D21, D22, D23, D24, D25, D26, D27, D28, D29, D3, D30, D32, D33, D34, D35, D36, D37, D38, D39, D4, D40, D41, D42, D43, D44, D45, D46, D47, D48, D49, D5, D50, D51, D52, D53, D54, D55, D56, D57, D58, D59, D6, D60, D61, D62, D63, D64, D65, D66, D67, D68, D69, D7, D8, D9, R1, R2, R3, R4, SW1, U1, X1: moved to B.Cu
- moved MH1 192.3 mm to (42.5, 56.0)
- moved C3 166.1 mm to (21.5, 91.0), turned to 0 degrees
- moved C4 161.7 mm to (26.5, 96.0), turned to 180 degrees
- moved C5 143.5 mm to (26.5, 98.5), turned to 180 degrees
- moved C7 142.9 mm to (26.5, 93.5), turned to 180 degrees
- moved C6 125.6 mm to (26.5, 91.0), turned to 180 degrees
- moved R2 60.4 mm to (126.7, 106.1), turned to 90 degrees
- moved U1 60.3 mm to (117.5, 111.3), turned to 90 degrees
- moved R3 44.2 mm to (117.5, 93.0), turned to 90 degrees
- moved C8 42.4 mm to (127.0, 121.3), turned to 0 degrees
- moved C1 39.7 mm to (105.5, 116.8), turned to 0 degrees
- moved X1 37.6 mm to (105.5, 113.3), turned to 90 degrees
- moved R4 36.2 mm to (136.6, 93.0), turned to 90 degrees
- moved C2 36.1 mm to (105.5, 109.8), turned to 180 degrees
- moved SW1 21.8 mm to (138.4, 113.3)
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- renumbered REF** to MH1
Connections:
- SPACE1 pad 1: /col4 -> /col9
- U1 pad 10: /col12 -> /row1
- U1 pad 11: /col13 -> /row2
- U1 pad 12: /col14 -> /row3
- U1 pad 18: /col15 -> Net-(U1-Pad18)
- U1 pad 22: Net-(U1-Pad22) -> /col1
- U1 pad 25: /col9 -> /col2
- U1 pad 26: /col8 -> /col3
- U1 pad 27: /col7 -> /col4
- U1 pad 28: /col6 -> /col5
- U1 pad 29: /col5 -> /col6
- U1 pad 30: /col4 -> /col7
- U1 pad 31: /col3 -> /col8
- U1 pad 32: /col2 -> /col9
- U1 pad 36: /col1 -> /col10
- U1 pad 37: /row5 -> /col11
- U1 pad 38: /row4 -> /col12
- U1 pad 39: /row3 -> /col13
- U1 pad 40: /row2 -> /col14
- U1 pad 41: /row1 -> /col15
- U1 pad 8: /col10 -> /row5
- U1 pad 9: /col11 -> /row4
Routing:
- net /row1: track 0.00 -> 405.9 mm, vias 0 -> 2
- net /row2: track 0.00 -> 363.6 mm, vias 0 -> 2
- net /row3: track 0.00 -> 343.9 mm, vias 0 -> 2
- net /row5: track 0.00 -> 305.6 mm, vias 0 -> 1
- net /row4: track 0.00 -> 296.4 mm, vias 0 -> 1
- net /col15: track 0.00 -> 281.2 mm
- net /col13: track 0.00 -> 272.0 mm
- net /col14: track 0.00 -> 266.0 mm
- net /col12: track 0.00 -> 246.5 mm
- net VCC: track 0.00 -> 237.6 mm, vias 0 -> 2
- net /col11: track 0.00 -> 232.8 mm
- net /col10: track 0.00 -> 185.8 mm
- net Net-(J1-Pad3): track 0.00 -> 181.9 mm
- net /col1: track 0.00 -> 181.3 mm
- net /col9: track 0.00 -> 179.9 mm, vias 0 -> 1
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- added copper zone on B.Cu, net GND
- added copper zone on F.Cu, net GND
Other:
- board outline added: 304.8 x 95.2 mm

Commit message: wow epic commit
Parts:
- renumbered PLUS1 to EQUAL1
