File: TKL2019/TKL2019.sch (KiCad schematic (older format))
At the start: 152 parts, among them J1 USB_mini_micro_B, SW1 SW_PUSH, U1 ATMEGA32U4, X1 XTAL_GND

Commit message: some footprints added
Parts:
- C1, C2, C3, C4, C5, C6, C7, C8: footprint (none) -> Capacitor_SMD:C_0805_2012Metric_Pad1.15x1.40mm_HandSolder
- D1, D2, D3, D4, D5, D6, D7, D8, D9: footprint (none) -> keyboard_parts:D_SOD123_axial
- D10, D11, D12, D13, D14, D15, D16, D17, D18, D19, D20, D21, D22, D23, D24, D25, D26, D27, D28, D29, D30, D32, D33, D34, D35, D36, D37, D38, D39, D40, D41, D42, D43, D44, D45, D46, D47, D48, D49, D50, D51, D52, D53, D54, D55, D56, D57, D58, D59, D60, D61, D62, D63, D64, D65, D66, D67, D68, D69: renamed from D?; footprint (none) -> keyboard_parts:D_SOD123_axial
- J1: footprint (none) -> keyboard_parts:USB_miniB_hirose_5S8
- R1, R2, R3, R4: footprint (none) -> Resistor_SMD:R_0805_2012Metric_Pad1.15x1.40mm_HandSolder
- SW1: footprint (none) -> Button_Switch_SMD:SW_SPST_TL3342
- U1: footprint (none) -> Package_QFP:TQFP-44_10x10mm_P0.8mm
- X1: footprint (none) -> oldstuff:crystal_FA238-TSX3225
- X2: renamed from X; footprint (none) -> Button_Switch_Keyboard:SW_Cherry_MX_6.25u_PCB
- renumbered A to A1, ALT to ALT1, ALT to ALT2, APOS to APOS1, B to B1, BACKSLASH to BACKSLASH1, BACKSPACE to BACKSPACE1, C to C9, CAPS to CAPS1, COMMA to COMMA1, CTRL to CTRL1, D to D31, DELETE to DELETE1, DOWN to DOWN1, E to E1, ENTER to ENTER1, ESC to ESC1, F to F1, FN to FN1, G to G1, H to H1, I to I1, J to J2, K to K1, L to L1, LCTRL to LCTRL1, LEFT to LEFT1, LKEY to LKEY1, LSHIFT to LSHIFT1, M to M1, MINUS to MINUS1, N to N1, O to O1, P to P1, PGDN to PGDN1, PGUP to PGUP1, PLUS to PLUS1, POINT to POINT1, POINTCOMMA to POINTCOMMA1, Q to Q1, R to R5, RIGHT to RIGHT1, RKEY to RKEY1, S to S1, SHIFT to SHIFT1, SLASH to SLASH1, SPACE to SPACE1, SUPER to SUPER1, T to T1, TAB to TAB1, TILDE to TILDE1, U to U2, UP to UP1, V to V1, W to W1, Y to Y1, Z to Z1

Commit message: sum progress
Parts:
- A1, APOS1, B1, C9, COMMA1, D31, DELETE1, DOWN1, E1, ESC1, F1, FN1, G1, H1, I1, J2, K1, L1, LEFT1, LKEY1, M1, MINUS1, N1, NO0, NO1, NO2, NO3, NO4, NO5, NO6, NO7, NO8, NO9, O1, P1, PGDN1, PGUP1, PLUS1, POINT1, POINTCOMMA1, Q1, R5, RIGHT1, RKEY1, S1, SLASH1, T1, TILDE1, U2, UP1, V1, W1, Y1, Z1: footprint (none) -> Button_Switch_Keyboard:SW_Cherry_MX_1.00u_Plate
- ALT1, CTRL1, SUPER1: footprint (none) -> Button_Switch_Keyboard:SW_Cherry_MX_1.25u_Plate
- BACKSLASH1, TAB1: footprint (none) -> Button_Switch_Keyboard:SW_Cherry_MX_1.50u_Plate
- BACKSPACE1: footprint (none) -> Button_Switch_Keyboard:SW_Cherry_MX_2.00u_Plate
- CAPS1: footprint (none) -> Button_Switch_Keyboard:SW_Cherry_MX_1.75u_Plate
- ENTER1, SHIFT1: footprint (none) -> Button_Switch_Keyboard:SW_Cherry_MX_2.25u_Plate
- RALT2: renamed from ALT2; footprint (none) -> Button_Switch_Keyboard:SW_Cherry_MX_1.00u_Plate
- RCTRL1: renamed from LCTRL1; footprint (none) -> Button_Switch_Keyboard:SW_Cherry_MX_1.00u_Plate
- RSHIFT1: renamed from LSHIFT1; footprint (none) -> Button_Switch_Keyboard:SW_Cherry_MX_1.75u_Plate
- SPACE1: footprint (none) -> Button_Switch_Keyboard:SW_Cherry_MX_6.25u_Plate
- X2: footprint Button_Switch_Keyboard:SW_Cherry_MX_6.25u_PCB -> Button_Switch_Keyboard:SW_Cherry_MX_1.00u_Plate

Commit message: a lot of progress
Parts:
- BACKSPACE1: footprint Button_Switch_Keyboard:SW_Cherry_MX_2.00u_Plate -> Button_Switch_Keyboard:SW_Cherry_MX_2.00u_PCB
- C1, C2, C3, C4, C5, C6, C7, C8: footprint Capacitor_SMD:C_0805_2012Metric_Pad1.15x1.40mm_HandSolder -> oldstuff:C_0805_HandSoldering
- ENTER1, SHIFT1: footprint Button_Switch_Keyboard:SW_Cherry_MX_2.25u_Plate -> Button_Switch_Keyboard:SW_Cherry_MX_2.25u_PCB
- R1, R2, R3, R4: footprint Resistor_SMD:R_0805_2012Metric_Pad1.15x1.40mm_HandSolder -> oldstuff:R_0805_HandSoldering
- SPACE1: footprint Button_Switch_Keyboard:SW_Cherry_MX_6.25u_Plate -> Button_Switch_Keyboard:SW_Cherry_MX_6.25u_PCB
Changed lines of the file:
@@
 F 0 "C2" H 2492 9446 50  0000 L CNN
 F 1 "22p" H 2492 9355 50  0000 L CNN
-F 2 "Capacitor_SMD:C_0805_2012Metric_Pad1.15x1.40mm_HandSolder" H 2400 9400 50  0001 C CNN
+F 2 "oldstuff:C_0805_HandSoldering" H 2400 9400 50  0001 C CNN
 F 3 "~" H 2400 9400 50  0001 C CNN
 	1    2400 9400
@@
 F 0 "C1" H 1892 9446 50  0000 L CNN
 F 1 "22p" H 1892 9355 50  0000 L CNN
-F 2 "Capacitor_SMD:C_0805_2012Metric_Pad1.15x1.40mm_HandSolder" H 1800 9400 50  0001 C CNN
+F 2 "oldstuff:C_0805_HandSoldering" H 1800 9400 50  0001 C CNN
 F 3 "~" H 1800 9400 50  0001 C CNN
 	1    1800 9400
@@
 F 0 "C6" H 6642 7846 50  0000 L CNN
 F 1 "0.1u" H 6642 7755 50  0000 L CNN
-F 2 "Capacitor_SMD:C_0805_2012Metric_Pad1.15x1.40mm_HandSolder" H 6550 7800 50  0001 C CNN
+F 2 "oldstuff:C_0805_HandSoldering" H 6550 7800 50  0001 C CNN
 F 3 "~" H 6550 7800 50  0001 C CNN
 	1    6550 7800
@@
 F 0 "C5" H 6992 7846 50  0000 L CNN
 F 1 "0.1u" H 6992 7755 50  0000 L CNN
-F 2 "Capacitor_SMD:C_0805_2012Metric_Pad1.15x1.40mm_HandSolder" H 6900 7800 50  0001 C CNN
+F 2 "oldstuff:C_0805_HandSoldering" H 6900 7800 50  0001 C CNN
 F 3 "~" H 6900 7800 50  0001 C CNN
 	1    6900 7800
@@
 F 0 "C4" H 7342 7846 50  0000 L CNN
 F 1 "0.1u" H 7342 7755 50  0000 L CNN
-F 2 "Capacitor_SMD:C_0805_2012Metric_Pad1.15x1.40mm_HandSolder" H 7250 7800 50  0001 C CNN
+F 2 "oldstuff:C_0805_HandSoldering" H 7250 7800 50  0001 C CNN
 F 3 "~" H 7250 7800 50  0001 C CNN
 	1    7250 7800
@@
 F 0 "C3" H 7692 7846 50  0000 L CNN
 F 1 "0.1u" H 7692 7755 50  0000 L CNN
-F 2 "Capacitor_SMD:C_0805_2012Metric_Pad1.15x1.40mm_HandSolder" H 7600 7800 50  0001 C CNN
+F 2 "oldstuff:C_0805_HandSoldering" H 7600 7800 50  0001 C CNN
 F 3 "~" H 7600 7800 50  0001 C CNN
 	1    7600 7800
@@
 F 0 "R1" V 2400 8100 50  0000 C TNN
 F 1 "10k" V 2600 8100 50  0000 C TNN
-F 2 "Resistor_SMD:R_0805_2012Metric_Pad1.15x1.40mm_HandSolder" V 2480 8100 50  0001 C CNN
+F 2 "oldstuff:R_0805_HandSoldering" V 2480 8100 50  0001 C CNN
 F 3 "~" H 2550 8100 50  0001 C CNN
 	1    2550 8100
@@
 F 0 "R2" V 6050 8350 50  0000 C TNN
 F 1 "10k" V 6250 8350 50  0000 C TNN
-F 2 "Resistor_SMD:R_0805_2012Metric_Pad1.15x1.40mm_HandSolder" V 6130 8350 50  0001 C CNN
+F 2 "oldstuff:R_0805_HandSoldering" V 6130 8350 50  0001 C CNN
 F 3 "~" H 6200 8350 50  0001 C CNN
 	1    6200 8350
@@
 F 0 "R3" V 3050 7350 50  0000 C TNN
 F 1 "22" V 3050 7550 50  0000 C TNN
-F 2 "Resistor_SMD:R_0805_2012Metric_Pad1.15x1.40mm_HandSolder" V 3030 7450 50  0001 C CNN
+F 2 "oldstuff:R_0805_HandSoldering" V 3030 7450 50  0001 C CNN
 F 3 "~" H 3100 7450 50  0001 C CNN
 	1    3100 7450
@@
 F 0 "R4" V 3050 7450 50  0000 C TNN
 F 1 "22" V 3050 7650 50  0000 C TNN
-F 2 "Resistor_SMD:R_0805_2012Metric_Pad1.15x1.40mm_HandSolder" V 3030 7550 50  0001 C CNN
+F 2 "oldstuff:R_0805_HandSoldering" V 3030 7550 50  0001 C CNN
 F 3 "~" H 3100 7550 50  0001 C CNN
 	1    3100 7550
@@
 F 0 "C8" V 3200 7800 50  0000 L CNN
 F 1 "1u" V 3200 7600 50  0000 L CNN
-F 2 "Capacitor_SMD:C_0805_2012Metric_Pad1.15x1.40mm_HandSolder" H 3250 7750 50  0001 C CNN
+F 2 "oldstuff:C_0805_HandSoldering" H 3250 7750 50  0001 C CNN
 F 3 "~" H 3250 7750 50  0001 C CNN
 	1    3250 7750
@@
 F 0 "BACKSPACE1" H 12250 1233 60  0000 C CNN
 F 1 "KEYSW" H 12250 900 60  0001 C CNN
-F 2 "Button_Switch_Keyboard:SW_Cherry_MX_2.00u_Plate" H 12250 1000 60  0001 C CNN
+F 2 "Button_Switch_Keyboard:SW_Cherry_MX_2.00u_PCB" H 12250 1000 60  0001 C CNN
 F 3 "" H 12250 1000 60  0000 C CNN
 	1    12250 1000
@@
 F 0 "ENTER1" H 11500 3033 60  0000 C CNN
 F 1 "KEYSW" H 11500 2700 60  0001 C CNN
-F 2 "Button_Switch_Keyboard:SW_Cherry_MX_2.25u_Plate" H 11500 2800 60  0001 C CNN
+F 2 "Button_Switch_Keyboard:SW_Cherry_MX_2.25u_PCB" H 11500 2800 60  0001 C CNN
 F 3 "" H 11500 2800 60  0000 C CNN
 	1    11500 2800
@@
 F 0 "SHIFT1" H 2500 3933 60  0000 C CNN
 F 1 "KEYSW" H 2500 3600 60  0001 C CNN
-F 2 "Button_Switch_Keyboard:SW_Cherry_MX_2.25u_Plate" H 2500 3700 60  0001 C CNN
+F 2 "Button_Switch_Keyboard:SW_Cherry_MX_2.25u_PCB" H 2500 3700 60  0001 C CNN
 F 3 "" H 2500 3700 60  0000 C CNN
 	1    2500 3700
@@
 F 0 "SPACE1" H 4750 4883 60  0000 C CNN
 F 1 "KEYSW" H 4750 4550 60  0001 C CNN
-F 2 "Button_Switch_Keyboard:SW_Cherry_MX_6.25u_Plate" H 4750 4650 60  0001 C CNN
+F 2 "Button_Switch_Keyboard:SW_Cherry_MX_6.25u_PCB" H 4750 4650 60  0001 C CNN
 F 3 "" H 4750 4650 60  0000 C CNN
 	1    4750 4650
@@
 F 0 "C7" H 6292 7846 50  0000 L CNN
 F 1 "4.7u" H 6292 7755 50  0000 L CNN
-F 2 "Capacitor_SMD:C_0805_2012Metric_Pad1.15x1.40mm_HandSolder" H 6200 7800 50  0001 C CNN
+F 2 "oldstuff:C_0805_HandSoldering" H 6200 7800 50  0001 C CNN
 F 3 "~" H 6200 7800 50  0001 C CNN
 	1    6200 7800

Commit message: changed some stuff
Parts:
- J1: footprint keyboard_parts:USB_miniB_hirose_5S8 -> SamacSys_Parts:1734035-2USB
Changed lines of the file:
@@
 F 0 "J1" H 1987 7791 60  0000 C CNN
 F 1 "USB_mini_micro_B" H 1950 7750 60  0001 C CNN
-F 2 "keyboard_parts:USB_miniB_hirose_5S8" H 2050 7500 60  0001 C CNN
+F 2 "SamacSys_Parts:1734035-2USB" H 2050 7500 60  0001 C CNN
 F 3 "" H 2050 7500 60  0000 C CNN
 	1    2100 7500

Commit message: bruh
Parts:
- added D70: LED, LED_THT:LED_D3.0mm, symbol Device:LED
- added R10, R6, R7, R8, R9: 22, oldstuff:R_0805_HandSoldering, symbol Device:R
Connections:
- wire segments 335 -> 336
- no-connect marks 6 -> 5
Other:
- moved on the sheet: D63, SPACE1
Changed lines of the file:
@@
 L keyboard_parts:KEYSW SPACE1
 U 1 1 5DFF0F5B
-P 4750 4650
-F 0 "SPACE1" H 4750 4883 60  0000 C CNN
-F 1 "KEYSW" H 4750 4550 60  0001 C CNN
-F 2 "Button_Switch_Keyboard:SW_Cherry_MX_6.25u_PCB" H 4750 4650 60  0001 C CNN
-F 3 "" H 4750 4650 60  0000 C CNN
-	1    4750 4650
+P 8500 4650
+F 0 "SPACE1" H 8500 4883 60  0000 C CNN
+F 1 "KEYSW" H 8500 4550 60  0001 C CNN
+F 2 "Button_Switch_Keyboard:SW_Cherry_MX_6.25u_PCB" H 8500 4650 60  0001 C CNN
+F 3 "" H 8500 4650 60  0000 C CNN
+	1    8500 4650
 	1    0    0    -1
 $EndComp
@@
 L keyboard_parts:D D63
 U 1 1 5DFF0F61
-P 4450 4950
-F 0 "D63" H 4322 4900 60  0000 R CNN
-F 1 "D" V 4600 4900 60  0001 C CNN
-F 2 "keyboard_parts:D_SOD123_axial" H 4450 4950 60  0001 C CNN
-F 3 "" H 4450 4950 60  0000 C CNN
-	1    4450 4950
-	-1   0    0    1
-$EndComp
-Wire Wire Line
-	4450 4650 4450 4800
-Wire Wire Line
-	4450 5000 4450 5150
+P 8200 4950
+F 0 "D63" H 8072 4900 60  0000 R CNN
+F 1 "D" V 8350 4900 60  0001 C CNN
+F 2 "keyboard_parts:D_SOD123_axial" H 8200 4950 60  0001 C CNN
+F 3 "" H 8200 4950 60  0000 C CNN
+	1    8200 4950
+	-1   0    0    1
+$EndComp
+Wire Wire Line
+	8200 4650 8200 4800
+Wire Wire Line
+	8200 5000 8200 5150
 $Comp
 L keyboard_parts:KEYSW RALT2
@@
 	2950 5150 3700 5150
 Connection ~ 3700 5150
-Wire Wire Line
-	3700 5150 4450 5150
-Connection ~ 4450 5150
 Connection ~ 8950 5150
 Wire Wire Line
@@
 Connection ~ 4300 3700
 Wire Wire Line
-	5050 3700 5050 4650
-Connection ~ 5050 3700
-Wire Wire Line
 	9550 3700 9550 4650
 Connection ~ 9550 3700
@@
 	13300 3700 13300 4650
 Connection ~ 13300 3700
-Wire Wire Line
-	4450 5150 8950 5150
 Wire Wire Line
 	3550 2800 3550 4650
@@
 Connection ~ 4300 4650
 Wire Wire Line
-	5050 4650 5050 5450
-Connection ~ 5050 4650
-Wire Wire Line
 	5800 3700 5800 5450
 Connection ~ 5800 3700
@@
 Connection ~ 8050 3700
 Wire Wire Line
-	8800 3700 8800 5450
+	8800 3700 8800 4650
 Connection ~ 8800 3700
 Wire Wire Line
@@
 Text Label 13300 5450 0    50   ~ 0
 col15
-Text Label 5650 7550 0    50   ~ 0
-row1
-Text Label 5650 7650 0    50   ~ 0
-row2
-Text Label 5650 7750 0    50   ~ 0
-row3
-Text Label 5650 7850 0    50   ~ 0
-row4
-Text Label 5650 7950 0    50   ~ 0
-row5
-Text Label 5650 8050 0    50   ~ 0
-col1
-Text Label 5650 8450 0    50   ~ 0
-col2
-Text Label 5650 8550 0    50   ~ 0
-col3
-Text Label 5650 8650 0    50   ~ 0
-col4
-Text Label 5650 8750 0    50   ~ 0
-col5
-Text Label 5650 8850 0    50   ~ 0
-col6
-Text Label 5650 8950 0    50   ~ 0
-col7
-Text Label 5650 9050 0    50   ~ 0
-col8
-Text Label 5650 9150 0    50   ~ 0
-col9
-Text Label 3500 7950 2    50   ~ 0
-col10
-Text Label 3500 8050 2    50   ~ 0
-col11
-Text Label 3500 8150 2    50   ~ 0
-col12
-Text Label 3500 8250 2    50   ~ 0
-col13
-Text Label 3500 8350 2    50   ~ 0
-col14
 $Comp
 L keyboard_parts:ATMEGA32U4 U1
@@
 	1    0    0    -1
 $EndComp
-Text Label 3500 8950 2    50   ~ 0
-col15
 $Comp
 L Device:C_Small C7
@@
 $EndComp
 NoConn ~ 3500 9050
-NoConn ~ 3500 9150
 NoConn ~ 3500 9250
-NoConn ~ 3500 9350
 NoConn ~ 5650 7450
+NoConn ~ 3500 8950
+Text Label 5650 7550 0    50   ~ 0
+col15
+Text Label 5650 7650 0    50   ~ 0
+col14
+Text Label 5650 7750 0    50   ~ 0
+col13
+Text Label 5650 7850 0    50   ~ 0
+col12
+Text Label 5650 7950 0    50   ~ 0
+col11
+Text Label 5650 8050 0    50   ~ 0
+col10
+Text Label 5650 8450 0    50   ~ 0
+col9
+Text Label 5650 8550 0    50   ~ 0
+col8
+Text Label 5650 8650 0    50   ~ 0
+col7
+Text Label 5650 8750 0    50   ~ 0
+col6
+Text Label 5650 8850 0    50   ~ 0
+col5
+Text Label 5650 8950 0    50   ~ 0
+col4
+Text Label 5650 9050 0    50   ~ 0
+col3
+Text Label 5650 9150 0    50   ~ 0
+col2
+Text Label 3500 9350 0    50   ~ 0
+col1
+Wire Wire Line
+	3700 5150 8200 5150
+Wire Wire Line
+	5050 3700 5050 5450
+Connection ~ 5050 3700
+Connection ~ 8200 5150
+Wire Wire Line
+	8200 5150 8950 5150
+Connection ~ 8800 4650
+Wire Wire Line
+	8800 4650 8800 5450
+Text Label 3500 7950 0    50   ~ 0
+row5
+Text Label 3500 8050 0    50   ~ 0
+row4
+Text Label 3500 8250 0    50   ~ 0
+row2
+Text Label 3500 8150 0    50   ~ 0
+row1
+Text Label 3500 8350 0    50   ~ 0
+row3
+$Comp
+L Device:LED D70
+U 1 1 5E4B97BE
+P 3800 10050
+F 0 "D70" V 3839 9933 50  0000 R CNN
+F 1 "LED" V 3748 9933 50  0000 R CNN
+F 2 "LED_THT:LED_D3.0mm" H 3800 10050 50  0001 C CNN
+F 3 "~" H 3800 10050 50  0001 C CNN
+	1    3800 10050
+	-1   0    0    1
+$EndComp
+$Comp
+L power:GND #PWR0118
+U 1 1 5E526F74
+P 3950 10050
+F 0 "#PWR0118" H 3950 9800 50  0001 C CNN
+F 1 "GND" H 3955 9877 50  0000 C CNN
+F 2 "" H 3950 10050 50  0001 C CNN
+F 3 "" H 3950 10050 50  0001 C CNN
+	1    3950 10050
+	0    -1   -1   0
+$EndComp
+$Comp
+L Device:R R8
+U 1 1 5E591F01
+P 3050 9900
+F 0 "R8" V 3000 9800 50  0000 C TNN
+F 1 "22" V 3000 10000 50  0000 C TNN
+F 2 "oldstuff:R_0805_HandSoldering" V 2980 9900 50  0001 C CNN
+F 3 "~" H 3050 9900 50  0001 C CNN
+	1    3050 9900
+	1    0    0    -1
+$EndComp
+$Comp
+L Device:R R7
+U 1 1 5E592520
+P 3050 9600
+F 0 "R7" V 3000 9500 50  0000 C TNN
+F 1 "22" V 3000 9700 50  0000 C TNN
+F 2 "oldstuff:R_0805_HandSoldering" V 2980 9600 50  0001 C CNN
+F 3 "~" H 3050 9600 50  0001 C CNN
+	1    3050 9600
+	1    0    0    -1
+$EndComp
+$Comp
+L Device:R R6
+U 1 1 5E59398F
+P 3050 9300
+F 0 "R6" V 3000 9200 50  0000 C TNN
+F 1 "22" V 3000 9400 50  0000 C TNN
+F 2 "oldstuff:R_0805_HandSoldering" V 2980 9300 50  0001 C CNN
+F 3 "~" H 3050 9300 50  0001 C CNN
+	1    3050 9300
+	1    0    0    -1
+$EndComp
+Wire Wire Line
+	3500 9150 3050 9150
+$Comp
+L Device:R R9
+U 1 1 5E5E196A
+P 3200 10050
+F 0 "R9" V 3150 9950 50  0000 C TNN
+F 1 "22" V 3150 10150 50  0000 C TNN
+F 2 "oldstuff:R_0805_HandSoldering" V 3130 10050 50  0001 C CNN
+F 3 "~" H 3200 10050 50  0001 C CNN
+	1    3200 10050
+	0    1    1    0
+$EndComp
+$Comp
+L Device:R R10
+U 1 1 5E5E22A5
+P 3500 10050
+F 0 "R10" V 3450 9950 50  0000 C TNN
+F 1 "22" V 3450 10150 50  0000 C TNN
+F 2 "oldstuff:R_0805_HandSoldering" V 3430 10050 50  0001 C CNN
+F 3 "~" H 3500 10050 50  0001 C CNN
+	1    3500 10050
+	0    1    1    0
+$EndComp
 $EndSCHEMATC

Commit message: wow epic commit
Parts:
- removed A1, APOS1, B1, C9, COMMA1, D31, DELETE1, DOWN1, E1, ESC1, F1, FN1, G1, H1, I1, J2, K1, L1, LEFT1, LKEY1, M1, MINUS1, N1, NO0, NO1, NO2, NO3, NO4, NO5, NO6, NO7, NO8, NO9, O1, P1, PGDN1, PGUP1, PLUS1, POINT1, POINTCOMMA1, Q1, R5, RALT2, RCTRL1, RIGHT1, RKEY1, S1, SLASH1, T1, TILDE1, U2, UP1, V1, W1, X2, Y1, Z1: KEYSW, Button_Switch_Keyboard:SW_Cherry_MX_1.00u_Plate, symbol keyboard_parts:KEYSW
- removed ALT1, CTRL1, SUPER1: KEYSW, Button_Switch_Keyboard:SW_Cherry_MX_1.25u_Plate, symbol keyboard_parts:KEYSW
- removed BACKSLASH1, TAB1: KEYSW, Button_Switch_Keyboard:SW_Cherry_MX_1.50u_Plate, symbol keyboard_parts:KEYSW
- removed BACKSPACE1: KEYSW, Button_Switch_Keyboard:SW_Cherry_MX_2.00u_PCB, symbol keyboard_parts:KEYSW
- removed C1, C2: 22p, oldstuff:C_0805_HandSoldering, symbol Device:C_Small
- removed C3, C4, C5, C6: 0.1u, oldstuff:C_0805_HandSoldering, symbol Device:C_Small
- removed C7: 4.7u, oldstuff:C_0805_HandSoldering, symbol Device:C_Small
- removed C8: 1u, oldstuff:C_0805_HandSoldering, symbol Device:C_Small
- removed CAPS1, RSHIFT1: KEYSW, Button_Switch_Keyboard:SW_Cherry_MX_1.75u_Plate, symbol keyboard_parts:KEYSW
- removed D1, D10, D11, D12, D13, D14, D15, D16, D17, D18, D19, D2, D20, D21, D22, D23, D24, D25, D26, D27, D28, D29, D3, D30, D32, D33, D34, D35, D36, D37, D38, D39, D4, D40, D41, D42, D43, D44, D45, D46, D47, D48, D49, D5, D50, D51, D52, D53, D54, D55, D56, D57, D58, D59, D6, D60, D61, D62, D63, D64, D65, D66, D67, D68, D69, D7, D8, D9: D, keyboard_parts:D_SOD123_axial, symbol keyboard_parts:D
- removed D70: LED, LED_THT:LED_D3.0mm, symbol Device:LED
- removed ENTER1, SHIFT1: KEYSW, Button_Switch_Keyboard:SW_Cherry_MX_2.25u_PCB, symbol keyboard_parts:KEYSW
- removed J1: USB_mini_micro_B, SamacSys_Parts:1734035-2USB, symbol keyboard_parts:USB_mini_micro_B
- removed R1, R2: 10k, oldstuff:R_0805_HandSoldering, symbol Device:R
- removed R10, R3, R4, R6, R7, R8, R9: 22, oldstuff:R_0805_HandSoldering, symbol Device:R
- removed SPACE1: KEYSW, Button_Switch_Keyboard:SW_Cherry_MX_6.25u_PCB, symbol keyboard_parts:KEYSW
- removed SW1: SW_PUSH, Button_Switch_SMD:SW_SPST_TL3342, symbol keyboard_parts:SW_PUSH
- removed U1: ATMEGA32U4, Package_QFP:TQFP-44_10x10mm_P0.8mm, symbol keyboard_parts:ATMEGA32U4
- removed X1: XTAL_GND, oldstuff:crystal_FA238-TSX3225, symbol keyboard_parts:XTAL_GND
Connections:
- net labels removed: GND, VCC, col1, col10, col11, col12, col13, col14, col15, col2, col3, col4, col5, col6, col7, col8, col9, row1, row2, row3, row4, row5
- wire segments 336 -> 0
- no-connect marks 5 -> 0

Commit message: fixed dead schematic
Parts:
- added A1, APOS1, B1, C9, COMMA1, D31, DELETE1, DOWN1, E1, ESC1, F1, FN1, G1, H1, I1, J2, K1, L1, LEFT1, LKEY1, M1, MINUS1, N1, NO0, NO1, NO2, NO3, NO4, NO5, NO6, NO7, NO8, NO9, O1, P1, PGDN1, PGUP1, PLUS1, POINT1, POINTCOMMA1, Q1, R5, RALT2, RCTRL1, RIGHT1, RKEY1, S1, SLASH1, T1, TILDE1, U2, UP1, V1, W1, X2, Y1, Z1: KEYSW, Button_Switch_Keyboard:SW_Cherry_MX_1.00u_Plate, symbol keyboard_parts:KEYSW
- added ALT1, CTRL1, SUPER1: KEYSW, Button_Switch_Keyboard:SW_Cherry_MX_1.25u_Plate, symbol keyboard_parts:KEYSW
- added BACKSLASH1, TAB1: KEYSW, Button_Switch_Keyboard:SW_Cherry_MX_1.50u_Plate, symbol keyboard_parts:KEYSW
- added BACKSPACE1: KEYSW, Button_Switch_Keyboard:SW_Cherry_MX_2.00u_PCB, symbol keyboard_parts:KEYSW
- added C1, C2: 22p, oldstuff:C_0805_HandSoldering, symbol Device:C_Small
- added C3, C4, C5, C6: 0.1u, oldstuff:C_0805_HandSoldering, symbol Device:C_Small
- added C7: 4.7u, oldstuff:C_0805_HandSoldering, symbol Device:C_Small
- added C8: 1u, oldstuff:C_0805_HandSoldering, symbol Device:C_Small
- added CAPS1, RSHIFT1: KEYSW, Button_Switch_Keyboard:SW_Cherry_MX_1.75u_Plate, symbol keyboard_parts:KEYSW
- added D1, D10, D11, D12, D13, D14, D15, D16, D17, D18, D19, D2, D20, D21, D22, D23, D24, D25, D26, D27, D28, D29, D3, D30, D32, D33, D34, D35, D36, D37, D38, D39, D4, D40, D41, D42, D43, D44, D45, D46, D47, D48, D49, D5, D50, D51, D52, D53, D54, D55, D56, D57, D58, D59, D6, D60, D61, D62, D63, D64, D65, D66, D67, D68, D69, D7, D8, D9: D, keyboard_parts:D_SOD123_axial, symbol keyboard_parts:D
- added D70: LED, LED_THT:LED_D3.0mm, symbol Device:LED
- added ENTER1, SHIFT1: KEYSW, Button_Switch_Keyboard:SW_Cherry_MX_2.25u_PCB, symbol keyboard_parts:KEYSW
- added J1: USB_mini_micro_B, SamacSys_Parts:1734035-2USB, symbol keyboard_parts:USB_mini_micro_B
- added R1, R2: 10k, oldstuff:R_0805_HandSoldering, symbol Device:R
- added R10, R3, R4, R6, R7, R8, R9: 22, oldstuff:R_0805_HandSoldering, symbol Device:R
- added SPACE1: KEYSW, Button_Switch_Keyboard:SW_Cherry_MX_6.25u_PCB, symbol keyboard_parts:KEYSW
- added SW1: SW_PUSH, Button_Switch_SMD:SW_SPST_TL3342, symbol keyboard_parts:SW_PUSH
- added U1: ATMEGA32U4, Package_QFP:TQFP-44_10x10mm_P0.8mm, symbol keyboard_parts:ATMEGA32U4
- added X1: XTAL_GND, oldstuff:crystal_FA238-TSX3225, symbol keyboard_parts:XTAL_GND
Connections:
- net labels added: GND, VCC, col1, col10, col11, col12, col13, col14, col15, col2, col3, col4, col5, col6, col7, col8, col9, row1, row2, row3, row4, row5
- wire segments 0 -> 336
- no-connect marks 0 -> 5
